Commit message: Update sim.urdf.xacro

File: exercise3/model/robots/sim.urdf.xacro (robot description, xacro)
@@ -90,5 +90,5 @@
     </link>
     <joint name="box3_joint" type="floating">
-        <origin xyz="0.75 0.3 0.026" rpy="0 0 0"/>
+        <origin xyz="0.55 -0.3 0.026" rpy="0 0 0"/>
         <parent link="base_link"/>
         <child link="box3"/>
