Commit message: Update sim.urdf.xacro
Muutin kuutioiden koon vastaamaan oikeeta

File: ltl_project/model/robots/sim.urdf.xacro (robot description, xacro)
@@ -18,5 +18,5 @@
         <visual>
             <geometry>
-                <box size="0.05 0.05 0.05"/>
+                <box size="0.025 0.025 0.025"/>
             </geometry>
             <material name="Cyan">
@@ -26,5 +26,5 @@
         <collision>
             <geometry>
-                <box size="0.05 0.05 0.05"/>
+                <box size="0.025 0.025 0.025"/>
             </geometry>
             <material name="Cyan">
@@ -46,5 +46,5 @@
         <visual>
             <geometry>
-                <box size="0.05 0.05 0.05"/>
+                <box size="0.025 0.025 0.025"/>
             </geometry>
             <material name="Cyan">
@@ -54,5 +54,5 @@
         <collision>
             <geometry>
-                <box size="0.05 0.05 0.05"/>
+                <box size="0.025 0.025 0.025"/>
             </geometry>
             <material name="Cyan">
@@ -74,5 +74,5 @@
         <visual>
             <geometry>
-                <box size="0.05 0.05 0.05"/>
+                <box size="0.025 0.025 0.025"/>
             </geometry>
             <material name="Cyan">
@@ -82,5 +82,5 @@
         <collision>
             <geometry>
-                <box size="0.05 0.05 0.05"/>
+                <box size="0.025 0.025 0.025"/>
             </geometry>
             <material name="Cyan">
@@ -102,5 +102,5 @@
         <visual>
             <geometry>
-                <box size="0.05 0.05 0.05"/>
+                <box size="0.025 0.025 0.025"/>
             </geometry>
             <material name="Cyan">
@@ -110,5 +110,5 @@
         <collision>
             <geometry>
-                <box size="0.05 0.05 0.05"/>
+                <box size="0.025 0.025 0.025"/>
             </geometry>
             <material name="Cyan">
